File: hardware/digital_input/digital_input.sch (KiCad schematic (older format))
At the start: 106 parts, among them IC1 PC817, IC10 PC817, IC11 PC817, IC12 PC817, IC13 PC817, IC14 PC817, IC15 PC817, IC16 PC817, IC2 PC817, IC3 PC817, IC4 PC817, IC5 PC817, IC6 PC817, IC7 PC817, IC8 PC817, IC9 PC817, K1 CONN_3_V, K2 CONN_3_V, K3 CONN_3_V, K4 CONN_3_V, K5 CONN_3_V, K6 CONN_3_V, P1 CONN_2_V, P3 CONN_6, U1 MCP23017

Commit message: Improved digital input circuit
Parts:
- removed K1, K2, K3: CONN_3_V, symbol CONN_3_V
- added P? (x8): CONN_2_V, symbol CONN_2_V
Connections:
- net at R1.1: now also P?.1 (P1)
- net at R2.1: now also P?.1 (P1)
- net at R3.1: now also P?.1 (P1)
- net at R4.1: now also P?.1 (P1)
- net at R5.1: now also P?.1 (P1)
- net at R6.1: now also P?.1 (P1)
- net at R7.1: now also P?.1 (P1)
- net at R8.1: now also P?.1 (P1)
- net at C8.2: now also D8.1 (A), IC8.2, P?.2 (P2)
- new net: C1.2, D1.1 (A), IC1.2, P?.2 (P2)
- new net: D2.1 (A), IC2.2, P?.2 (P2)
- new net: D3.1 (A), IC3.2, P?.2 (P2)
- new net: D4.1 (A), IC4.2, P?.2 (P2)
- new net: D5.1 (A), IC5.2, P?.2 (P2)
- new net: D6.1 (A), IC6.2, P?.2 (P2)
- new net: D7.1 (A), IC7.2, P?.2 (P2)
Other:
- note added: "Isolated 24VDC supply to external digital input sources"
- note removed: "24V supply to external sensors and switches."
Changed lines of the file:
@@
 LIBS:contrib
 LIBS:valves
+LIBS:borniers
 LIBS:digital_input-cache
 EELAYER 27 0
@@
 Sheet 1 1
 Title "Digitalt inngangskort"
-Date "3 jun 2015"
+Date "5 jun 2015"
 Rev "1"
 Comp "Haustveit elektro"
@@
 	1    0    0    -1
 $EndComp
-$Comp
-L CONN_3_V K1
-U 1 1 556E105C
-P 900 1500
-F 0 "K1" H 800 1750 50  0000 C CNN
-F 1 "CONN_3_V" H 900 1690 40  0000 C CNN
-F 2 "" H 900 1500 60  0000 C CNN
-F 3 "" H 900 1500 60  0000 C CNN
-	1    900  1500
-	-1   0    0    -1
-$EndComp
-$Comp
-L CONN_3_V K2
-U 1 1 556E1069
-P 900 2000
-F 0 "K2" H 800 2250 50  0000 C CNN
-F 1 "CONN_3_V" H 900 2190 40  0000 C CNN
-F 2 "" H 900 2000 60  0000 C CNN
-F 3 "" H 900 2000 60  0000 C CNN
-	1    900  2000
-	-1   0    0    -1
-$EndComp
-$Comp
-L CONN_3_V K3
-U 1 1 556E106F
-P 900 2500
-F 0 "K3" H 800 2750 50  0000 C CNN
-F 1 "CONN_3_V" H 900 2690 40  0000 C CNN
-F 2 "" H 900 2500 60  0000 C CNN
-F 3 "" H 900 2500 60  0000 C CNN
-	1    900  2500
-	-1   0    0    -1
-$EndComp
 Wire Wire Line
 	4450 1400 4600 1400
@@
 Connection ~ 3950 2350
 Wire Wire Line
-	2300 1950 2700 1950
+	1250 1950 2700 1950
 Wire Wire Line
 	3250 2350 4600 2350
@@
 Connection ~ 3950 2900
 Wire Wire Line
-	2200 2500 2700 2500
+	1250 2500 2700 2500
 Wire Wire Line
 	3250 2900 4600 2900
@@
 Connection ~ 3950 3450
 Wire Wire Line
-	2100 3050 2700 3050
+	1250 3050 2700 3050
 Wire Wire Line
 	3250 3450 4600 3450
@@
 Connection ~ 3950 4000
 Wire Wire Line
-	2000 3600 2700 3600
-Wire Wire Line
 	3250 4000 4600 4000
 Wire Wire Line
@@
 Connection ~ 3950 4550
 Wire Wire Line
-	1900 4150 2700 4150
-Wire Wire Line
 	3250 4550 4600 4550
 Wire Wire Line
@@
 Connection ~ 3950 5050
 Wire Wire Line
-	1800 4650 2700 4650
-Wire Wire Line
 	3250 5050 4600 5050
 Wire Wire Line
@@
 	4600 5600 4600 5400
 Connection ~ 3950 5600
-Wire Wire Line
-	1700 5200 2700 5200
-Wire Wire Line
-	1600 5600 4600 5600
 Wire Wire Line
 	5300 5400 5350 5400
@@
 	14550 9550 14550 9700
 Connection ~ 14550 10150
-Wire Wire Line
-	3250 1800 3250 5600
-Connection ~ 3250 2350
-Connection ~ 3250 2900
-Connection ~ 3250 3450
-Connection ~ 3250 4000
-Connection ~ 3250 4550
-Connection ~ 3250 5050
-Connection ~ 3250 5600
 Connection ~ 3600 1400
 Connection ~ 3600 1800
-Wire Wire Line
-	2300 1950 2300 1500
-Wire Wire Line
-	2300 1500 1250 1500
-Wire Wire Line
-	1250 1600 2200 1600
-Wire Wire Line
-	2200 1600 2200 2500
-Wire Wire Line
-	1250 1900 2100 1900
-Wire Wire Line
-	2100 1900 2100 3050
-Wire Wire Line
-	1250 2000 2000 2000
-Wire Wire Line
-	2000 2000 2000 3600
-Wire Wire Line
-	1250 2100 1900 2100
-Wire Wire Line
-	1900 2100 1900 4150
-Wire Wire Line
-	1250 2400 1800 2400
-Wire Wire Line
-	1800 2400 1800 4650
-Wire Wire Line
-	1250 2500 1700 2500
-Wire Wire Line
-	1700 2500 1700 5200
-Wire Wire Line
-	1600 5600 1600 2600
-Wire Wire Line
-	1600 2600 1250 2600
 $Comp
 L PC817 IC9
@@
 Wire Wire Line
 	13500 9650 13500 10150
-Text Notes 13400 8950 0    60   ~ 0
-24V supply to external sensors and switches.
+Text Notes 11450 8850 0    100  ~ 0
+Isolated 24VDC supply to external digital input sources
 Text Notes 10500 1700 0    60   ~ 0
 Address selection jumpers.
+$Comp
+L CONN_2_V P?
+U 1 1 5571AEF3
+P 900 1500
+F 0 "P?" H 820 1725 40  0000 C CNN
+F 1 "CONN_2_V" H 870 1680 40  0000 C CNN
+F 2 "" H 900 1500 60  0000 C CNN
+F 3 "" H 900 1500 60  0000 C CNN
+	1    900  1500
+	-1   0    0    -1
+$EndComp
+Wire Wire Line
+	1250 1600 3250 1600
+Wire Wire Line
+	1250 5200 2700 5200
+Wire Wire Line
+	1250 4650 2700 4650
+Wire Wire Line
+	1250 4150 2700 4150
+Wire Wire Line
+	1250 3600 2700 3600
+$Comp
+L CONN_2_V P?
+U 1 1 5571B056
+P 900 2050
+F 0 "P?" H 820 2275 40  0000 C CNN
+F 1 "CONN_2_V" H 870 2230 40  0000 C CNN
+F 2 "" H 900 2050 60  0000 C CNN
+F 3 "" H 900 2050 60  0000 C CNN
+	1    900  2050
+	-1   0    0    -1
+$EndComp
+$Comp
+L CONN_2_V P?
+U 1 1 5571B05C
+P 900 2600
+F 0 "P?" H 820 2825 40  0000 C CNN
+F 1 "CONN_2_V" H 870 2780 40  0000 C CNN
+F 2 "" H 900 2600 60  0000 C CNN
+F 3 "" H 900 2600 60  0000 C CNN
+	1    900  2600
+	-1   0    0    -1
+$EndComp
+$Comp
+L CONN_2_V P?
+U 1 1 5571B062
+P 900 3150
+F 0 "P?" H 820 3375 40  0000 C CNN
+F 1 "CONN_2_V" H 870 3330 40  0000 C CNN
+F 2 "" H 900 3150 60  0000 C CNN
+F 3 "" H 900 3150 60  0000 C CNN
+	1    900  3150
+	-1   0    0    -1
+$EndComp
+$Comp
+L CONN_2_V P?
+U 1 1 5571B1C0
+P 900 3700
+F 0 "P?" H 820 3925 40  0000 C CNN
+F 1 "CONN_2_V" H 870 3880 40  0000 C CNN
+F 2 "" H 900 3700 60  0000 C CNN
+F 3 "" H 900 3700 60  0000 C CNN
+	1    900  3700
+	-1   0    0    -1
+$EndComp
+$Comp
+L CONN_2_V P?
+U 1 1 5571B1C6
+P 900 4250
+F 0 "P?" H 820 4475 40  0000 C CNN
+F 1 "CONN_2_V" H 870 4430 40  0000 C CNN
+F 2 "" H 900 4250 60  0000 C CNN
+F 3 "" H 900 4250 60  0000 C CNN
+	1    900  4250
+	-1   0    0    -1
+$EndComp
+$Comp
+L CONN_2_V P?
+U 1 1 5571B1CC
+P 900 4750
+F 0 "P?" H 820 4975 40  0000 C CNN
+F 1 "CONN_2_V" H 870 4930 40  0000 C CNN
+F 2 "" H 900 4750 60  0000 C CNN
+F 3 "" H 900 4750 60  0000 C CNN
+	1    900  4750
+	-1   0    0    -1
+$EndComp
+$Comp
+L CONN_2_V P?
+U 1 1 5571B1D2
+P 900 5300
+F 0 "P?" H 820 5525 40  0000 C CNN
+F 1 "CONN_2_V" H 870 5480 40  0000 C CNN
+F 2 "" H 900 5300 60  0000 C CNN
+F 3 "" H 900 5300 60  0000 C CNN
+	1    900  5300
+	-1   0    0    -1
+$EndComp
+Wire Wire Line
+	3250 1600 3250 1800
+Wire Wire Line
+	1250 2150 3250 2150
+Wire Wire Line
+	3250 2150 3250 2350
+Wire Wire Line
+	1250 2700 3250 2700
+Wire Wire Line
+	3250 2700 3250 2900
+Wire Wire Line
+	1250 3250 3250 3250
+Wire Wire Line
+	3250 3250 3250 3450
+Wire Wire Line
+	1250 3800 3250 3800
+Wire Wire Line
+	3250 3800 3250 4000
+Wire Wire Line
+	1250 4350 3250 4350
+Wire Wire Line
+	3250 4350 3250 4550
+Wire Wire Line
+	1250 4850 3250 4850
+Wire Wire Line
+	3250 4850 3250 5050
+Wire Wire Line
+	1250 5400 3250 5400
+Wire Wire Line
+	3250 5400 3250 5600
+Wire Wire Line
+	3250 5600 4600 5600
+Connection ~ 3600 5600
 $EndSCHEMATC

Commit message: Improved digital output card with modbus controller
Parts:
- removed K4, K5, K6: CONN_3_V, symbol CONN_3_V
- added P10, P11, P12, P13, P14, P15, P16, P9: CONN_2_V, symbol CONN_2_V
- C1, C9: value 0u1 -> 100nF
- C10, C11, C12, C13, C14, C15, C16, C2, C3, C4, C5, C6, C7, C8: value C -> 100nF
- R10, R11, R12, R13, R14, R15, R16, R2, R3, R4, R5, R6, R7, R8: value R -> 2k4
- gave numbers to parts that had none: 12
- renumbered D33 to D34, P1 to P17, P3 to P18, R18 to R17, R19 to R18, R20 to R19, R17 to R21
Connections:
- net at R9.1: now also P9.1 (P1)
- net at R10.1: now also P10.1 (P1)
- net at R11.1: now also P11.1 (P1)
- net at R12.1: now also P12.1 (P1)
- net at R13.1: now also P13.1 (P1)
- net at R14.1: now also P14.1 (P1)
- net at R15.1: now also P15.1 (P1)
- net at R16.1: now also P16.1 (P1)
- net at C16.2: now also D16.1 (A), IC16.2, P16.2 (P2)
- new net: C9.2, D9.1 (A), IC9.2, P9.2 (P2)
- new net: D10.1 (A), IC10.2, P10.2 (P2)
- new net: D11.1 (A), IC11.2, P11.2 (P2)
- new net: D12.1 (A), IC12.2, P12.2 (P2)
- new net: D13.1 (A), IC13.2, P13.2 (P2)
- new net: D14.1 (A), IC14.2, P14.2 (P2)
- new net: D15.1 (A), IC15.2, P15.2 (P2)
