File: hardware/digital_output/digital_output.sch (KiCad schematic (older format))
At the start: 132 parts, among them P1 CONN_2_V, P10 CONN_6, P11 CONN_2_V, P12 CONN_2_V, P13 CONN_2_V, P14 CONN_2_V, P15 CONN_2_V, P16 CONN_2_V, P17 CONN_2_V, P18 CONN_2_V, P2 CONN_2_V, P3 CONN_2_V, P4 CONN_2_V, P5 CONN_2_V, P6 CONN_2_V, P7 CONN_2_V, P8 CONN_2_V, Q1 BC548, Q10 BC548, Q11 BC548, Q12 BC548, Q13 BC548, Q14 BC548, Q15 BC548, Q16 BC548, Q2 BC548, Q3 BC548, Q4 BC548, Q5 BC548, Q6 BC548, Q7 BC548, Q8 BC548, Q9 BC548, U1 74LS595, U2 74LS595

Commit message: Improved digital output card with modbus controller
Parts:
- removed D10, D13, D14, D17, D18, D21, D22: LED, ~, symbol LED
- removed D2, D27, D28, D3, D31, D32, D4, D7, D8: DIODE, ~, symbol DIODE
- removed P10: CONN_6, symbol CONN_6
- removed P13, P18, P2: CONN_2_V, symbol CONN_2_V
- removed Q1, Q10, Q11, Q12, Q13, Q14, Q15, Q16, Q2, Q3, Q4, Q5, Q6, Q7, Q8, Q9: BC548, TO92, symbol BC548
- removed R19, R20, R21, R22, R23, R24: 4k7, ~, symbol R
- removed R2, R25, R26, R27, R28, R29, R30, R31, R32: 500R, ~, symbol R
- removed RL2: RM50-XX11, symbol RM50-XX11
- removed U1, U2: 74LS595, ~, symbol 74LS595
- removed VR2: VR, ~, symbol VR
- added C1, C2, C4, C6: 100n, ~, symbol C
- added C3, C5: 22p, ~, symbol C
- added D1, D10, D13, D14, D17, D18, D21, D22, D9: DIODE, ~, symbol DIODE
- added D27, D28, D3, D31, D34, D7, D8: LED, ~, symbol LED
- added D32, D33: TVS_BIPOL, symbol TVS_BIPOL
- added F1, F10, F11, F12, F13, F14, F15, F16, F17, F18, F2, F3, F4, F5, F6, F7, F8, F9: PPTC, symbol PPTC
- added IC1: ATMEGA16-P, DIL40, symbol ATMEGA16-P
- added IC2: MAX485, ~, symbol MAX485
- added P1, P10, P9: CONN_2_V, symbol CONN_2_V
- added P13: CONN_5X2, symbol CONN_5X2
- added R1: 1k, ~, symbol R
- added RL1: RM50-XX11, symbol RM50-XX11
- added SW1: SW_RESET, ~, symbol SW_PUSH
- added U1, U2, U3: ULN2003, symbol ULN2003
- added VR1: VR, ~, symbol VR
- added X1: 16MHz, ~, symbol CRYSTAL
- R10, R11, R12, R13, R14, R15, R16, R17: value 4k7 -> 1k
- R18: value 4k7 -> 0R
- R2: renamed from R1; value 500R -> 1k
- R3, R4, R5, R6, R7, R8: value 500R -> 1k
- R9: value 4k7 -> 10k
- gave numbers to parts that had none: 1
- renumbered D1 to D2, D9 to D4, P1 to P2, RL1 to RL2, VR1 to VR2
Connections:
- net labels added: +24V, CPU_RESET, REL10, REL11, REL12, REL13, REL14, REL15, REL16, REL9, RS485_A, RS485_B, TCK, TDI, TDO, TMS, Y0.0, Y0.1, Y0.2, Y0.3, Y0.4, Y0.5, Y0.6, Y0.7, Y1.0, Y1.1, Y1.2, Y1.3, Y1.4, Y1.5, Y1.6, Y1.7
- wire segments 433 -> 427
- no-connect marks 17 -> 36
Other:
- note added: "Atmega 16 modbus slave"
- note added: "External diodes might be redundant."
- note added: "JTAG"
- note added: "May be replased by a short if the circuit is protected externally."
- note added: "PPTC(Polymer Positive Temerature Coefficient) fuses must have a rating of 250V 5A."
- note added: "ULN2003 Transistor arrays"
- note added: "ULN2003 has built in flyback diodes."
- moved on the sheet: D2, D4, K1, P2, R2, VR2
